Commit message: add

File: myrobot/urdf/myrobot.xacro (robot description, xacro)
@@ -78,5 +78,5 @@
  </link>
   <joint type="continuous" name="right_wheel_hinge">
-    <origin xyz="0 0.15 0" rpy="0 0 0"/>
+    <origin xyz="0 -0.15 0" rpy="0 0 0"/>
     <child link="link_right_wheel"/>
     <parent link="chassis"/>
@@ -107,5 +107,5 @@
  </link>
   <joint type="continuous" name="left_wheel_hinge">
-    <origin xyz="0 -0.15 0" rpy="0 0 0"/>
+    <origin xyz="0 0.15 0" rpy="0 0 0"/>
     <child link="link_left_wheel"/>
     <parent link="chassis"/>

Commit message: fixed sunk

File: myrobot/urdf/myrobot.xacro (robot description, xacro)
@@ -4,5 +4,5 @@
 <xacro:include filename="$(find myrobot)/urdf/myrobot.gazebo" />
   <joint name="robot_footprint_joint" type="fixed">
-    <origin xyz="0 0 0" rpy="0 0 0" />
+    <origin xyz="0 0 0.1" rpy="0 0 0" />
     <parent link="robot_footprint"/>
     <child link="chassis" />
